File: Line Generator/Line Generator.sch (KiCad schematic (older format))
At the start: 22 parts, among them J1 Conn_01x04, Q1 BS170F, Q2 BCV46, Q3 BCV46, Q4 BS170F

Commit message: Track widths increased
Parts:
- R2, R3, R6, R7: footprint Resistor_SMD:R_0603_1608Metric_Pad1.05x0.95mm_HandSolder -> Resistor_SMD:R_0805_2012Metric_Pad1.15x1.40mm_HandSolder
Changed lines of the file:
@@
 EESchema Schematic File Version 4
-EELAYER 30 0
+LIBS:Line Generator-cache
+EELAYER 29 0
 EELAYER END
 $Descr A4 11693 8268
@@
 F 0 "R3" H 4995 2146 50  0000 L CNN
 F 1 "4K7" H 4995 2055 50  0000 L CNN
-F 2 "Resistor_SMD:R_0603_1608Metric_Pad1.05x0.95mm_HandSolder" V 4855 2100 50  0001 C CNN
+F 2 "Resistor_SMD:R_0805_2012Metric_Pad1.15x1.40mm_HandSolder" V 4855 2100 50  0001 C CNN
 F 3 "~" H 4925 2100 50  0001 C CNN
 	1    4925 2100
@@
 F 0 "R2" H 4375 1500 50  0000 L CNN
 F 1 "100K" H 4300 1400 50  0000 L CNN
-F 2 "Resistor_SMD:R_0603_1608Metric_Pad1.05x0.95mm_HandSolder" V 4480 1450 50  0001 C CNN
+F 2 "Resistor_SMD:R_0805_2012Metric_Pad1.15x1.40mm_HandSolder" V 4480 1450 50  0001 C CNN
 F 3 "~" H 4550 1450 50  0001 C CNN
 	1    4550 1450
@@
 F 0 "R6" H 7045 2146 50  0000 L CNN
 F 1 "4K7" H 7045 2055 50  0000 L CNN
-F 2 "Resistor_SMD:R_0603_1608Metric_Pad1.05x0.95mm_HandSolder" V 6905 2100 50  0001 C CNN
+F 2 "Resistor_SMD:R_0805_2012Metric_Pad1.15x1.40mm_HandSolder" V 6905 2100 50  0001 C CNN
 F 3 "~" H 6975 2100 50  0001 C CNN
 	1    6975 2100
@@
 F 0 "R7" H 7175 1475 50  0000 L CNN
 F 1 "100K" H 7100 1375 50  0000 L CNN
-F 2 "Resistor_SMD:R_0603_1608Metric_Pad1.05x0.95mm_HandSolder" V 7280 1425 50  0001 C CNN
+F 2 "Resistor_SMD:R_0805_2012Metric_Pad1.15x1.40mm_HandSolder" V 7280 1425 50  0001 C CNN
 F 3 "~" H 7350 1425 50  0001 C CNN
 	1    7350 1425
