File: 2D Top Board/2D Top Board.kicad_pcb (KiCad board)
At the start: 2 copper layers, 84.9 x 59.4 mm, 35 parts, among them J1 Conn_02x15_Top_Bottom, J10 Conn_01x04, J2 Conn_02x15_Top_Bottom, J3 Conn_02x15_Top_Bottom, J4 Conn_01x02, J5 Conn_01x02, J6 647676-2, J7 Conn_01x06, J8 Conn_01x04, J9 Conn_01x05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

Commit message: Updated top board
Parts:
- removed Fan1, Fan2, Fan3, Fan4: MountingHole_3.2mm_M3_ISO14580, MountingHole:MountingHole_3.2mm_M3_ISO14580
- removed R1, R2: 1K, Resistor_SMD:R_0603_1608Metric_Pad1.05x0.95mm_HandSolder
Connections:
- J4 pad 2: Net-(J4-Pad2) -> GND
- J5 pad 2: Net-(J5-Pad2) -> GND
Routing:
- net +3V3: track 206.1 -> 177.1 mm
- net Net-(J5-Pad2): track 4.38 -> 0.00 mm
- net Net-(J4-Pad2): track 4.38 -> 0.00 mm
- added copper zone on B.Cu, net GND
Other:
- outline, holes or cut-outs redrawn
- board text added: "2D Top Board"
