File: 2D Top Board/2D Top Board.sch (KiCad schematic (older format))
At the start: 31 parts, among them J1 Conn_02x15_Top_Bottom, J10 Conn_01x04, J2 Conn_02x15_Top_Bottom, J3 Conn_02x15_Top_Bottom, J4 Conn_01x02, J5 Conn_01x02, J6 647676-2, J7 Conn_01x06, J8 Conn_01x04, J9 Conn_01x05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

Commit message: Updated top board
Parts:
- removed R1, R2: 1K, Resistor_SMD:R_0603_1608Metric_Pad1.05x0.95mm_HandSolder, symbol Device:R
Connections:
- net GND: now also J4.2 (Pin_2), J5.2 (Pin_2)
Changed lines of the file:
@@
 Wire Wire Line
 	3675 3400 3875 3400
-$Comp
-L power:+3.3V #PWR0130
-U 1 1 5EDD1D09
-P 3500 3500
-F 0 "#PWR0130" H 3500 3350 50  0001 C CNN
-F 1 "+3.3V" V 3500 3725 50  0000 C CNN
-F 2 "" H 3500 3500 50  0001 C CNN
-F 3 "" H 3500 3500 50  0001 C CNN
-	1    3500 3500
-	0    -1   -1   0
-$EndComp
-$Comp
-L Device:R R2
-U 1 1 5EDD2036
-P 3700 3500
-F 0 "R2" V 3775 3450 50  0000 L CNN
-F 1 "1K" V 3700 3425 50  0000 L CNN
-F 2 "Resistor_SMD:R_0603_1608Metric_Pad1.05x0.95mm_HandSolder" V 3630 3500 50  0001 C CNN
-F 3 "~" H 3700 3500 50  0001 C CNN
-	1    3700 3500
-	0    1    1    0
-$EndComp
-$Comp
-L Device:R R1
-U 1 1 5EDD3F26
-P 3700 3000
-F 0 "R1" V 3775 2950 50  0000 L CNN
-F 1 "1K" V 3700 2925 50  0000 L CNN
-F 2 "Resistor_SMD:R_0603_1608Metric_Pad1.05x0.95mm_HandSolder" V 3630 3000 50  0001 C CNN
-F 3 "~" H 3700 3000 50  0001 C CNN
-	1    3700 3000
-	0    1    1    0
-$EndComp
-Wire Wire Line
-	3850 3500 3875 3500
-Wire Wire Line
-	3500 3500 3550 3500
-$Comp
-L power:+3.3V #PWR0131
-U 1 1 5EE0E970
-P 3475 3000
-F 0 "#PWR0131" H 3475 2850 50  0001 C CNN
-F 1 "+3.3V" V 3475 3225 50  0000 C CNN
-F 2 "" H 3475 3000 50  0001 C CNN
-F 3 "" H 3475 3000 50  0001 C CNN
-	1    3475 3000
-	0    -1   -1   0
-$EndComp
-Wire Wire Line
-	3850 3000 3875 3000
-Wire Wire Line
-	3550 3000 3475 3000
+Wire Wire Line
+	3675 3500 3875 3500
+Wire Wire Line
+	3675 3000 3875 3000
 Text Notes 3375 2750 0    50   ~ 0
 Reed Switch
@@
 Wire Wire Line
 	5800 5625 6675 5625
+$Comp
+L power:GND #PWR0130
+U 1 1 5E6B1D9F
+P 3675 3000
+F 0 "#PWR0130" H 3675 2750 50  0001 C CNN
+F 1 "GND" V 3675 2775 50  0000 C CNN
+F 2 "" H 3675 3000 50  0000 C CNN
+F 3 "" H 3675 3000 50  0000 C CNN
+	1    3675 3000
+	0    1    1    0
+$EndComp
+$Comp
+L power:GND #PWR0131
+U 1 1 5E6BDA82
+P 3675 3500
+F 0 "#PWR0131" H 3675 3250 50  0001 C CNN
+F 1 "GND" V 3675 3275 50  0000 C CNN
+F 2 "" H 3675 3500 50  0000 C CNN
+F 3 "" H 3675 3500 50  0000 C CNN
+	1    3675 3500
+	0    1    1    0
+$EndComp
 $EndSCHEMATC
