File: New Top Board/Top Board.sch (KiCad schematic (older format))
At the start: 35 parts, among them J1 Conn_01x04, J10 Conn_01x04, J11 Conn_01x02, J12 Conn_01x02, J13 RJE392881400, J14 RJE392881400, J2 68611514122, J3 Conn_01x06, J4 Conn_01x04, J5 Screw_Terminal_01x02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

Commit message: updated library paths
Parts:
- J13, J14: symbol RJE392881400:RJE392881400 -> Top-Board-rescue:RJE392881400-RJE392881400
- J2: symbol 68611514122:68611514122 -> Top-Board-rescue:68611514122-68611514122
- U2: symbol dk_Logic-Signal-Switches-Multiplexers-Decoders:LTC4314 -> Top-Board-rescue:LTC4314-dk_Logic-Signal-Switches-Multiplexers-Decoders
- U3, U7: symbol dk_Logic-Signal-Switches-Multiplexers-Decoders:FSA642 -> Top-Board-rescue:FSA642-dk_Logic-Signal-Switches-Multiplexers-Decoders
- U5: symbol MC14555BCPG:MC14555BCPG -> Top-Board-rescue:MC14555BCPG-MC14555BCPG
Changed lines of the file:
@@
 NoConn ~ 10050 5925
 $Comp
-L dk_Logic-Signal-Switches-Multiplexers-Decoders:FSA642 U7
+L Top-Board-rescue:FSA642-dk_Logic-Signal-Switches-Multiplexers-Decoders U7
 U 1 1 5E3D8DE0
 P 10350 4725
@@
 NoConn ~ 8400 5925
 $Comp
-L dk_Logic-Signal-Switches-Multiplexers-Decoders:FSA642 U3
+L Top-Board-rescue:FSA642-dk_Logic-Signal-Switches-Multiplexers-Decoders U3
 U 1 1 5E3DCDB0
 P 8700 4725
@@
 Connection ~ 7450 3875
 $Comp
-L dk_Logic-Signal-Switches-Multiplexers-Decoders:LTC4314 U2
+L Top-Board-rescue:LTC4314-dk_Logic-Signal-Switches-Multiplexers-Decoders U2
 U 1 1 5E41218A
 P 7100 4975
@@
 	6500 5175 6800 5175
 $Comp
-L MC14555BCPG:MC14555BCPG U5
+L Top-Board-rescue:MC14555BCPG-MC14555BCPG U5
 U 1 1 5E4D62A0
 P 9675 2275
@@
 NoConn ~ 1375 3000
 $Comp
-L 68611514122:68611514122 J2
+L Top-Board-rescue:68611514122-68611514122 J2
 U 1 1 5EC3F9CE
 P 3600 1600
@@
 	1275 1500 1375 1500
 $Comp
-L RJE392881400:RJE392881400 J13
+L Top-Board-rescue:RJE392881400-RJE392881400 J13
 U 1 1 5ECBCF3A
 P 4425 800
@@
 $EndComp
 $Comp
-L RJE392881400:RJE392881400 J14
+L Top-Board-rescue:RJE392881400-RJE392881400 J14
 U 1 1 5ECBF9F6
 P 6875 775

Commit message: Corrected MC14555BDG to include a GND connection
Parts:
- removed U2: LTC4314, digikey-footprints:SOP65P777X199-20N, symbol Top-Board-rescue:LTC4314-dk_Logic-Signal-Switches-Multiplexers-Decoders
- added U2: LTC4314, digikey-footprints:SOP65P777X199-20N, symbol dk_Logic-Signal-Switches-Multiplexers-Decoders:LTC4314
Changed lines of the file:
@@
-	1    0    0    -1
-$EndComp
-Connection ~ 7450 3875
-$Comp
-L Top-Board-rescue:LTC4314-dk_Logic-Signal-Switches-Multiplexers-Decoders U2
-U 1 1 5E41218A
-P 7100 4975
-F 0 "U2" H 7528 5153 60  0000 L CNN
-F 1 "LTC4314" V 7400 4975 60  0000 L CNN
-F 2 "digikey-footprints:SOP65P777X199-20N" H 7550 5275 60  0001 L CNN
-F 3 "http://www.ti.com/general/docs/suppproductinfo.tsp?distId=10&gotoUrl=http%3A%2F%2Fwww.ti.com%2Flit%2Fgpn%2Ftca9548a" H 7550 5375 60  0001 L CNN
-F 4 "LTC4314" H 7550 5475 60  0001 L CNN "MPN"
-F 5 "Integrated Circuits (ICs)" H 7550 5575 60  0001 L CNN "Category"
-F 6 "Logic - Signal Switches, Multiplexers, Decoders" H 7550 5675 60  0001 L CNN "Family"
-F 7 "Pin Selectable, 4 Channel, 2 wire multiplexer" H 7550 5775 60  0001 L CNN "Description"
-F 8 "Linear Technology" H 7550 5875 60  0001 L CNN "Manufacturer"
-F 9 "Active" H 7550 5975 60  0001 L CNN "Status"
-	1    7100 4975
 	1    0    0    -1
 $EndComp
@@
 Text GLabel 5725 4375 0    50   Input ~ 10
 CAMERASDA
-Wire Wire Line
-	7400 5900 7400 5825
-$Comp
-L power:GND #PWR0121
-U 1 1 5E3187FE
-P 7400 5900
-F 0 "#PWR0121" H 7400 5650 50  0001 C CNN
-F 1 "GND" V 7400 5675 50  0000 C CNN
-F 2 "" H 7400 5900 50  0000 C CNN
-F 3 "" H 7400 5900 50  0000 C CNN
-	1    7400 5900
-	1    0    0    -1
-$EndComp
 Wire Wire Line
 	3825 7400 4000 7400
@@
 Wire Wire Line
 	4000 7500 3825 7500
+$Comp
+L dk_Logic-Signal-Switches-Multiplexers-Decoders:LTC4314 U2
+U 1 1 5F64C318
+P 7100 4975
+F 0 "U2" H 7528 5153 60  0000 L CNN
+F 1 "LTC4314" V 7575 4700 60  0000 L CNN
+F 2 "digikey-footprints:SOP65P777X199-20N" H 7550 5275 60  0001 L CNN
+F 3 "http://www.ti.com/general/docs/suppproductinfo.tsp?distId=10&gotoUrl=http%3A%2F%2Fwww.ti.com%2Flit%2Fgpn%2Ftca9548a" H 7550 5375 60  0001 L CNN
+F 4 "LTC4314" H 7550 5475 60  0001 L CNN "MPN"
+F 5 "Integrated Circuits (ICs)" H 7550 5575 60  0001 L CNN "Category"
+F 6 "Logic - Signal Switches, Multiplexers, Decoders" H 7550 5675 60  0001 L CNN "Family"
+F 7 "Pin Selectable, 4 Channel, 2 wire multiplexer" H 7550 5775 60  0001 L CNN "Description"
+F 8 "Linear Technology" H 7550 5875 60  0001 L CNN "Manufacturer"
+F 9 "Active" H 7550 5975 60  0001 L CNN "Status"
+	1    7100 4975
+	1    0    0    -1
+$EndComp
+Connection ~ 7450 3875
+$Comp
+L power:GND #PWR0121
+U 1 1 5F64D888
+P 7400 5900
+F 0 "#PWR0121" H 7400 5650 50  0001 C CNN
+F 1 "GND" H 7405 5727 50  0000 C CNN
+F 2 "" H 7400 5900 50  0001 C CNN
+F 3 "" H 7400 5900 50  0001 C CNN
+	1    7400 5900
+	1    0    0    -1
+$EndComp
+Wire Wire Line
+	7400 5825 7400 5900
 $EndSCHEMATC
